File: 3_Elektronik/KiCad/power.kicad_sch (KiCad schematic)
At the start: 0 parts

Commit message: fix: :bug: rename usb_pd to generic power schematic
Parts:
- added C19: 1µF, Capacitor_SMD:C_0603_1608Metric, symbol Device:C_Small
- added C25: 10µF, Capacitor_SMD:C_0603_1608Metric, symbol Device:C_Small
- added C3: 150 µF, AUXSPACE:CP_Wurth_WCAP-ASLL-D6.3L5.5, symbol AUXSPACE:D6.3L5.5_865060243005
- added C4: 100nF, Capacitor_SMD:C_0603_1608Metric, symbol Device:C_Small
- added D10: 8240136, AUXSPACE:WE-TVS_SOT143-4L, symbol AUXSPACE:WE-TVS-HS_SOT143-4L_8240136
- added D11: SMAJ22A, AUXSPACE:WE-TVS_SMAJ22A, symbol AUXSPACE:WE-TVSP_DO-214AC_400W_UNI
- added D12: 824094024, AUXSPACE:WE-TVS_824094024_SOT23-3L, symbol AUXSPACE:SOT23-3L_824094024
- added J7: 629722000214, AUXSPACE:J_Wurth_WR-USB_629722000214, symbol AUXSPACE:629722000214
- added Q2: DMP3099L, Package_TO_SOT_SMD:SOT-23, symbol Transistor_FET:DMP3099L
- added R30, R33: 5,1k, Resistor_SMD:R_0603_1608Metric, symbol Device:R
- added R32: 100k, Resistor_SMD:R_0603_1608Metric, symbol Device:R
- added R34: 10k, Resistor_SMD:R_0603_1608Metric, symbol Device:R
- added R4: 11k, Resistor_SMD:R_0603_1608Metric, symbol Device:R_Small
- added R6: 2,7k, Resistor_SMD:R_0603_1608Metric, symbol Device:R_Small
- added U2: TPS7B8601QDDARQ1, AUXSPACE:Texas_R-PDSO-G8_EP2.95x4.9mm_Mask2.4x3.1mm_ThermalVias, symbol AUXSPACE:TPS7B8601QDDARQ1
- added U8: CH224A, AUXSPACE:ESSOP-10-1EP_3.9x5.0mm_P1mm_EP2.1x3.3mm, symbol CH224A:CH224A
Connections:
- new net: C19.2, C3.1, R32.2, U8.1 (VHV), U8.8 (VBUS)
- new net: R34.2, U8.10 (PG)
- new net: R4.2, R6.1, U2.2 (FB)
- new net: Q2.1 (G), R34.1
- new net +3V3: C25.1, R4.1, U2.1 (OUT)
- new net CC1: D12.1 (I/O1), J7.A5 (CC1), R33.1, U8.7 (CC1)
- new net CC2: D12.2 (I/O2), J7.B5 (CC2), R30.1, U8.6 (CC2)
- new net GND: C19.1, C25.2, C3.2, C4.2, D10.1, D11.2, D12.3 (GND), J7.A1 (GND), J7.A12 (GND1), J7.B1 (GND3), J7.B12 (GND2), J7.S1 (SHIELD), J7.S2 (SHIELD), J7.S3 (SHIELD), J7.S4 (SHIELD), R30.2, R33.2, R6.2, U2.3 (NC), U2.4 (NC), U2.5 (GND), U2.6 (NC), U2.9 (Thermal_Pad), U8.11 (GND), U8.2 (CFG2/SCL), U8.3 (CFG3/SDA), U8.9 (CFG1)
- new net USB_D+: D10.2, J7.A6 (D+1), J7.B6 (D+2), U8.4 (DP)
- new net USB_D-: D10.3, J7.A7 (D-1), J7.B7 (D-2), U8.5 (DM)
- new net VBus_direct: C4.1, Q2.3 (D), U2.7 (EN), U2.8 (IN)
- new net Vusb: D11.1, J7.A4 (VBUS), J7.A9 (VBUS1), J7.B4 (VBUS3), J7.B9 (VBUS2), Q2.2 (S), R32.1
- no-connect marks 0 -> 3
Other:
- note added: "3V3 Power Source"
- note added: "9V"
- note added: "CFG1 CFG2 CFG3 Voltage ------------------ 0 0 0 9V 0 0 1 12V 0 1 1 20V 0 1 0 28V 1 X X 5V"
- note added: "Nanjing Qinheng CH224A"
- note added: "POWER"
- note added: "Protection"
- note added: "TSV Diode"
- note added: "USB 2.0 compat"
- note added: "USB D+/D-"
- note added: "USB PD"
- note added: "USB Type-C"
- note added: "for USB CC Pins"
