File: 3_Elektronik/KiCad/mcu.kicad_sch (KiCad schematic)
At the start: 22 parts, among them J5 Conn_01x04_Pin, SW2 434331013822, SW3 434331013822, U4 ESP32-S3-WROOM-1

Commit message: fix: move D11 in current path
This commit also fixes the messed-up footprint of J1
Parts:
- J5: footprint (none) -> Connector_PinHeader_2.54mm:PinHeader_1x04_P2.54mm_Vertical
Changed lines of the file:
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@@
 			)
 		)
-		(property "Footprint" ""
+		(property "Footprint" "Connector_PinHeader_2.54mm:PinHeader_1x04_P2.54mm_Vertical"
 			(at 135.89 62.23 0)
 			(hide yes)

Commit message: build: :wrench: swap baro with meas ms5607
Use the MS5607 since it can measure up to ~30km above sea level.
The DPS was only able to measure up to ~9km.
Connections:
- net BARO_INT: no longer names the net of U4.24 (IO47)
- no-connect marks 3 -> 4
Changed lines of the file:
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@@
 		(at 109.22 82.55)
 	)
+	(no_connect
+		(at 109.22 107.95)
+	)
 	(wire
 		(pts
@@
 		(pts
 			(xy 59.69 95.25) (xy 78.74 95.25)
-		)
-		(stroke
-			(width 0)
-			(type default)
-		)
-	)
-	(wire
-		(pts
-			(xy 109.22 107.95) (xy 129.54 107.95)
 		)
 		(stroke
@@
 		)
 	)
-	(hierarchical_label "BARO_INT"
-		(shape passive)
-		(at 129.54 107.95 0)
-		(effects
-			(font
-				(size 1.27 1.27)
-			)
-			(justify left)
-		)
-	)
